File: circuits/rev_a.sch (EAGLE design)
At the start: 5 parts

Commit message: Finished a rev a, but it's enormous.
Parts:
- added D1, D2, D3: APA102-2020, SparkFun-LED:APA102-2020
- added R3: 10k, adafruit:R-US_R0603
- added R4, R5, R6, R7, R8, R9: (no value), adafruit:R-US_R0603
- added X1: ENCODER_ANO, custom:ENCODER_ANO
- MCU: value TEENSY_4.0-ANALOG-DEPIN -> TEENSY_4.0-NOBOTTOM; device Teensy-4.0:TEENSY_4.0-ANALOG-DEPIN -> Teensy-4.0:TEENSY_4.0-NOBOTTOM
Connections:
- new net N$1: MCU.6, R9.1, X1.S5
- new net N$10: D2.DO, D3.DI
- new net N$11: D2.CO, D3.CI
- new net N$12: D1.CI, MCU.13/SCK
- new net N$13: D1.DI, MCU.11/MOSI
- new net N$2: MCU.5, R8.1, X1.S4
- new net N$3: MCU.4, R7.1, X1.S3
- new net N$4: MCU.3, R6.1, X1.S2
- new net N$5: MCU.2, R5.1, X1.1
- new net N$6: MCU.1/TX1, R4.1, X1.B
- new net N$7: MCU.0/RX1, R3.2, X1.A
- new net N$8: D1.DO, D2.DI
- new net N$9: D1.CO, D2.CI
- net +3V3: now also D1.VCC, D2.VCC, D3.VCC, R3.1, R4.2, R5.2, R6.2, R7.2, R8.2, R9.2
- net GND: now also D1.GND, D2.GND, D3.GND, X1.COMA, X1.COM_B
Other:
- moved on the sheet: R1, R2
