File: circuits/rev_d.brd (EAGLE design)
At the start: 61 x 58 mm, 16 parts, among them X1 ENCODER_ANO

Commit message: Working through feature suggestions.
Connections:
- net N$1: now also MCU.8; no longer MCU.6
- net N$2: now also MCU.7; no longer MCU.5
- net N$3: now also MCU.6; no longer MCU.4/CANRX
- net N$4: now also MCU.5; no longer MCU.3/CANTX
- net N$5: now also MCU.4/CANRX; no longer MCU.2
- net N$6: now also MCU.3/CANTX; no longer MCU.1/TX
- net N$7: now also MCU.2; no longer MCU.0/RX
Routing:
- net +3V3: track 185.9 -> 0.00 mm, vias 5 -> 0
- net S2: track 89.9 -> 0.00 mm
- net N$12: track 70.5 -> 0.00 mm, vias 1 -> 0
- net HOR2: track 60.8 -> 0.00 mm
- net N$13: track 60.0 -> 0.00 mm, vias 1 -> 0
- net N$7: track 57.0 -> 0.00 mm
- net N$4: track 47.8 -> 0.00 mm
- net VERT2: track 39.7 -> 0.00 mm
- net HOR1: track 39.5 -> 0.00 mm
- net N$5: track 38.6 -> 0.00 mm
- net N$1: track 35.5 -> 0.00 mm
- net S1: track 33.8 -> 0.00 mm
- net N$3: track 32.9 -> 0.00 mm, vias 1 -> 0
- net N$6: track 30.7 -> 0.00 mm
- net VERT1: track 23.9 -> 0.00 mm
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