File: circuits/macro_rat.brd (EAGLE design)
At the start: 62 x 82 mm, 14 parts, among them K0 KEY_LED_CHOC_ONESIDERIGHT_HAND, K1 KEY_LED_CHOC_ONESIDERIGHT_HAND, K2 KEY_LED_CHOC_ONESIDERIGHT_HAND, K3 KEY_LED_CHOC_ONESIDERIGHT_HAND, K4 KEY_LED_CHOC_ONESIDERIGHT_HAND, K5 KEY_LED_CHOC_ONESIDERIGHT_HAND

Commit message: Lots of progress in hardware and software.
Parts:
- D1, D2, D3: device SparkFun-LED:APA102-2020 -> custom:APA102-2020
- moved R2 4.51 mm to (35.5, 12.4)
Connections:
- net +3V3: now also K0.PULLUP_V, K0.PULLUP_VIA, K1.PULLUP_V, K1.PULLUP_VIA, K2.PULLUP_V, K2.PULLUP_VIA, K3.PULLUP_V, K3.PULLUP_VIA, K4.PULLUP_V, K4.PULLUP_VIA, K5.PULLUP_V, K5.PULLUP_VIA
- net 5V: now also D1.5V_VIA, D2.5V_VIA, D3.5V_VIA
- net GND: now also D1.GND_VIA, D2.GND_VIA, D3.GND_VIA
- net K0: now also K0.OUT_UP
- net K1: now also K1.OUT_UP
- net K2: now also K2.OUT_UP
- net K3: now also K3.OUT_UP
- net K4: now also K4.OUT_UP
- net K5: now also K5.OUT_UP
Routing:
- net +3V3: track 108.9 -> 232.1 mm
- net K3: track 46.6 -> 51.4 mm
- net K5: track 48.7 -> 52.0 mm
- net K2: track 49.3 -> 52.0 mm
- net N$17: track 60.5 -> 63.1 mm
- net S2: track 31.5 -> 29.0 mm
- net K4: track 43.2 -> 45.7 mm
- net K1: track 31.1 -> 33.6 mm
- net K0: track 35.3 -> 37.7 mm
- net N$15: track 69.2 -> 66.8 mm
- net N$18: track 64.3 -> 63.0 mm
- net N$13: track 14.0 -> 12.9 mm
- net 5V: track 222.3 -> 223.1 mm, vias 3 -> 0
- net N$16: track 67.6 -> 67.0 mm
- net N$4: track 17.6 -> 18.1 mm
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Other:
- outline, holes or cut-outs redrawn
