File: circuits/macro_rat.sch (EAGLE design)
At the start: 14 parts, among them K0 KEY_LED_CHOC_ONESIDERIGHT_HAND, K1 KEY_LED_CHOC_ONESIDERIGHT_HAND, K2 KEY_LED_CHOC_ONESIDERIGHT_HAND, K3 KEY_LED_CHOC_ONESIDERIGHT_HAND, K4 KEY_LED_CHOC_ONESIDERIGHT_HAND, K5 KEY_LED_CHOC_ONESIDERIGHT_HAND

Commit message: Lots of progress in hardware and software.
Parts:
- D1, D2, D3: device SparkFun-LED:APA102-2020 -> custom:APA102-2020
Connections:
- net +3V3: now also K0.PULLUP, K1.PULLUP, K2.PULLUP, K3.PULLUP, K4.PULLUP, K5.PULLUP
Changed lines of the file:
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@@
 <part name="R1" library="adafruit" library_urn="urn:adsk.eagle:library:420" deviceset="R-US_" device="R0603" package3d_urn="urn:adsk.eagle:package:6240565/1" value="10k"/>
 <part name="R2" library="adafruit" library_urn="urn:adsk.eagle:library:420" deviceset="R-US_" device="R0603" package3d_urn="urn:adsk.eagle:package:6240565/1" value="10k"/>
-<part name="D1" library="SparkFun-LED" deviceset="APA102" device="-2020"/>
-<part name="D2" library="SparkFun-LED" deviceset="APA102" device="-2020"/>
-<part name="D3" library="SparkFun-LED" deviceset="APA102" device="-2020"/>
+<part name="D1" library="custom" deviceset="APA102" device="-2020"/>
+<part name="D2" library="custom" deviceset="APA102" device="-2020"/>
+<part name="D3" library="custom" deviceset="APA102" device="-2020"/>
 <part name="GND4" library="supply1" library_urn="urn:adsk.eagle:library:371" deviceset="GND" device=""/>
 <part name="K0" library="custom" deviceset="KEY_LED_CHOC_ONESIDE" device="RIGHT_HAND" value="KEY_LED_CHOC_ONESIDERIGHT_HAND"/>
@@
 <wire x1="101.6" y1="55.88" x2="101.6" y2="63.5" width="0.1524" layer="91"/>
 </segment>
+<segment>
+<pinref part="K0" gate="G$1" pin="PULLUP"/>
+<pinref part="K1" gate="G$1" pin="PULLUP"/>
+<wire x1="142.24" y1="-43.18" x2="182.88" y2="-43.18" width="0.1524" layer="91"/>
+<pinref part="K2" gate="G$1" pin="PULLUP"/>
+<wire x1="182.88" y1="-43.18" x2="223.52" y2="-43.18" width="0.1524" layer="91"/>
+<junction x="182.88" y="-43.18"/>
+<label x="203.2" y="-43.18" size="1.778" layer="95"/>
+</segment>
+<segment>
+<pinref part="K3" gate="G$1" pin="PULLUP"/>
+<pinref part="K4" gate="G$1" pin="PULLUP"/>
+<wire x1="142.24" y1="-88.9" x2="182.88" y2="-88.9" width="0.1524" layer="91"/>
+<pinref part="K5" gate="G$1" pin="PULLUP"/>
+<wire x1="182.88" y1="-88.9" x2="223.52" y2="-88.9" width="0.1524" layer="91"/>
+<junction x="182.88" y="-88.9"/>
+<label x="193.04" y="-88.9" size="1.778" layer="95"/>
+</segment>
 </net>
 <net name="S2" class="0">
@@
 <segment>
 <pinref part="K0" gate="G$1" pin="5V"/>
-<wire x1="139.7" y1="-40.64" x2="180.34" y2="-40.64" width="0.1524" layer="91"/>
+<wire x1="137.16" y1="-40.64" x2="177.8" y2="-40.64" width="0.1524" layer="91"/>
 <label x="187.96" y="-40.64" size="1.778" layer="95"/>
 <pinref part="K1" gate="G$1" pin="5V"/>
-<wire x1="180.34" y1="-40.64" x2="220.98" y2="-40.64" width="0.1524" layer="91"/>
-<junction x="180.34" y="-40.64"/>
+<wire x1="177.8" y1="-40.64" x2="218.44" y2="-40.64" width="0.1524" layer="91"/>
+<junction x="177.8" y="-40.64"/>
 <pinref part="K2" gate="G$1" pin="5V"/>
 </segment>
 <segment>
-<wire x1="139.7" y1="-86.36" x2="180.34" y2="-86.36" width="0.1524" layer="91"/>
+<wire x1="137.16" y1="-86.36" x2="177.8" y2="-86.36" width="0.1524" layer="91"/>
 <label x="185.42" y="-86.36" size="1.778" layer="95"/>
 <pinref part="K3" gate="G$1" pin="5V"/>
 <pinref part="K4" gate="G$1" pin="5V"/>
-<wire x1="180.34" y1="-86.36" x2="220.98" y2="-86.36" width="0.1524" layer="91"/>
-<junction x="180.34" y="-86.36"/>
+<wire x1="177.8" y1="-86.36" x2="218.44" y2="-86.36" width="0.1524" layer="91"/>
+<junction x="177.8" y="-86.36"/>
 <pinref part="K5" gate="G$1" pin="5V"/>
 </segment>
