File: circuits/simple_rat.brd (EAGLE design)
At the start: 62 x 40 mm, 8 parts

Commit message: Lots of progress in hardware and software.
Parts:
- D1, D2, D3: device SparkFun-LED:APA102-2020 -> custom:APA102-2020
- moved R2 5.50 mm to (35.8, 13.4)
Connections:
- net 5V: now also D1.5V_VIA, D2.5V_VIA, D3.5V_VIA
- net GND: now also D1.GND_VIA, D2.GND_VIA, D3.GND_VIA
Routing:
- net +3V3: track 108.9 -> 103.4 mm
- net S2: track 31.5 -> 27.3 mm
- net N$13: track 14.0 -> 12.6 mm
- net 5V: track 95.7 -> 94.4 mm, vias 3 -> 0
- net GND: track 2.70 -> 2.96 mm, vias 3 -> 0
Other:
- outline, holes or cut-outs redrawn
