File: circuits/simple_rat.sch (EAGLE design)
At the start: 8 parts

Commit message: Lots of progress in hardware and software.
Parts:
- D1, D2, D3: device SparkFun-LED:APA102-2020 -> custom:APA102-2020
Changed lines of the file:
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@@
 <part name="R1" library="adafruit" library_urn="urn:adsk.eagle:library:420" deviceset="R-US_" device="R0603" package3d_urn="urn:adsk.eagle:package:6240565/1" value="10k"/>
 <part name="R2" library="adafruit" library_urn="urn:adsk.eagle:library:420" deviceset="R-US_" device="R0603" package3d_urn="urn:adsk.eagle:package:6240565/1" value="10k"/>
-<part name="D1" library="SparkFun-LED" deviceset="APA102" device="-2020"/>
-<part name="D2" library="SparkFun-LED" deviceset="APA102" device="-2020"/>
-<part name="D3" library="SparkFun-LED" deviceset="APA102" device="-2020"/>
+<part name="D1" library="custom" deviceset="APA102" device="-2020"/>
+<part name="D2" library="custom" deviceset="APA102" device="-2020"/>
+<part name="D3" library="custom" deviceset="APA102" device="-2020"/>
 <part name="GND4" library="supply1" library_urn="urn:adsk.eagle:library:371" deviceset="GND" device=""/>
 </parts>
